File: KiCad Files/new_synth/new_synth/new_synth.sch (KiCad schematic (older format))
At the start: 28 parts

Commit message: Adding new synth with transistors as switches
Parts:
- removed J?: Conn_ARM_JTAG_SWD_10, Connector_PinHeader_1.27mm:PinHeader_2x05_P1.27mm_Vertical_SMD, symbol Connector:Conn_ARM_JTAG_SWD_10
- removed R?: 10K, symbol Device:R
- removed U?: CD74HCT4066QPWRQ1, PW14, symbol new_synth-rescue:CD74HCT4066QPWRQ1-Synth
- removed U?: STM32F072RBTx, Package_QFP:LQFP-64_10x10mm_P0.5mm, symbol MCU_ST_STM32F0:STM32F072RBTx
- added C?: C_100nF, symbol Device:C
- added J?: Conn_ARM_JTAG_SWD_10, Connector_PinHeader_1.27mm:PinHeader_2x05_P1.27mm_Vertical_SMD, symbol Connector:Conn_ARM_JTAG_SWD_10
- added R5: R, symbol Device:R
- added U2: STM32F072RBTx, Package_QFP:LQFP-64_10x10mm_P0.5mm, symbol MCU_ST_STM32F0:STM32F072RBTx
- R2: renamed from R?; footprint (none) -> Resistor_SMD:R_0805_2012Metric_Pad1.15x1.40mm_HandSolder
- R4: renamed from R?; value 1K -> R; footprint (none) -> Resistor_SMD:R_0805_2012Metric_Pad1.15x1.40mm_HandSolder
- RV1, RV2, RV3: renamed from RV?; value 5M -> R_POT
- gave numbers to parts that had none: 14
Connections:
- net labels added: SWCLK, SWDCLK, SWDIO
- net labels removed: C12, C13, C5, D, R
- wire segments 69 -> 48
Other:
- moved on the sheet: D1, D2, D4, R4, RV4, U4C
