File: Synth - Final/new_synth_transistor.kicad_pcb (KiCad board)
At the start: 2 copper layers, 6 parts, among them J1 Conn_ARM_JTAG_SWD_10, Q1 2N3904, Q2 2N3904, Q3 2N3904, Q4 2N3904, U4 STM32F072RBTx

Commit message: Add PCB
Parts:
- added C1: C_0.1uF, Capacitor_SMD:C_0805_2012Metric, F.Cu at (164.3, 95.8)
- added C10: C_22pF, Capacitor_SMD:C_0805_2012Metric, F.Cu at (161.0, 75.9)
- added C11: C_0.1uF, Capacitor_SMD:C_0805_2012Metric, F.Cu at (175.0, 82.7)
- added C12: C_0.1uF, Capacitor_SMD:C_0805_2012Metric, F.Cu at (173.8, 97.7)
- added C13: C_0.1uF, Capacitor_SMD:C_0805_2012Metric, F.Cu at (166.0, 82.6)
- added C14: C_0.1uF, Capacitor_SMD:C_0805_2012Metric, F.Cu at (123.8, 83.2)
- added C17: C_2.2uF, Capacitor_SMD:C_0805_2012Metric, F.Cu at (199.3, 80.7)
- added C2: C_0.1uF, Capacitor_SMD:C_0805_2012Metric, F.Cu at (188.7, 94.3)
- added C3: C_0.1uF, Capacitor_SMD:C_0805_2012Metric, F.Cu at (142.9, 92.0)
- added C4: C_0.1uF, Capacitor_SMD:C_0805_2012Metric, F.Cu at (181.2, 94.3)
- added C5: C_0.1uF, Capacitor_SMD:C_0805_2012Metric, F.Cu at (129.8, 90.7)
- added C6: C_0.1uF, Capacitor_SMD:C_0805_2012Metric, F.Cu at (177.9, 70.6)
- added C7: C_22pF, Capacitor_SMD:C_0805_2012Metric, F.Cu at (161.1, 71.2)
- added C8: C_0.1uF, Capacitor_SMD:C_0805_2012Metric, F.Cu at (161.0, 78.8)
- added C9: C_0.1uF, Capacitor_SMD:C_0805_2012Metric, F.Cu at (166.0, 67.4)
- added CR1: BAT60JFILM, BAT60JFILM:BAT60JFILM, F.Cu at (190.1, 76.1)
- added CR2: BAT60JFILM, BAT60JFILM:BAT60JFILM, F.Cu at (180.0, 64.5)
- added CR3: BAT60JFILM, BAT60JFILM:BAT60JFILM, F.Cu at (216.1, 68.5)
- added CR4: BAT60JFILM, BAT60JFILM:BAT60JFILM, F.Cu at (194.7, 72.8)
- added D1: LED, Diode_SMD:D_0805_2012Metric, F.Cu at (140.7, 58.3)
- added D2: LED, Diode_SMD:D_0805_2012Metric, F.Cu at (167.1, 57.9)
- added D3: LED, Diode_SMD:D_0805_2012Metric, F.Cu at (162.8, 57.9)
- added D4: LED, Diode_SMD:D_0805_2012Metric, F.Cu at (158.7, 57.9)
- added D5: LED, Diode_SMD:D_0805_2012Metric, F.Cu at (154.6, 57.9)
- added J2: Conn_01x07_Male, Connector_PinHeader_2.54mm:PinHeader_1x07_P2.54mm_Vertical, F.Cu at (202.3, 85.9)
- added J3: Conn_01x07_Male, Connector_PinHeader_2.54mm:PinHeader_1x07_P2.54mm_Vertical, F.Cu at (154.1, 52.5)
- added J4: Conn_01x07_Male, Connector_PinHeader_2.54mm:PinHeader_1x07_P2.54mm_Vertical, F.Cu at (138.9, 98.8)
- added J5: USB_B, AU-Y1007:ASSMANN_AU-Y1007, F.Cu at (120.8, 54.5)
- added J6: Conn_ARM_JTAG_SWD_10, Connector_PinHeader_1.27mm:PinHeader_2x05_P1.27mm_Vertical_SMD, F.Cu at (173.0, 59.7)
- added J7: UJ2-MIBH-4-SMT-TR, digikey-footprints:USB_Micro_B_Male_UJ2-MIBH-4-SMT-TR, F.Cu at (210.8, 62.0)
- added R1: R_200, Resistor_SMD:R_0805_2012Metric, F.Cu at (144.4, 58.3)
- added R10: R_1K, Resistor_SMD:R_0805_2012Metric, F.Cu at (217.1, 73.0)
- added R11: R_4K, Resistor_SMD:R_0805_2012Metric, F.Cu at (219.9, 75.7)
- added R12: R_200, Resistor_SMD:R_0805_2012Metric, F.Cu at (194.0, 65.6)
- added R13: R_499K, Resistor_SMD:R_0805_2012Metric, F.Cu at (211.7, 68.0)
- added R14: R_1K, Resistor_SMD:R_0805_2012Metric, F.Cu at (193.5, 76.0)
- added R15: R_200, Resistor_SMD:R_0805_2012Metric, F.Cu at (200.4, 65.3)
- added R16: R_200, Resistor_SMD:R_0805_2012Metric, F.Cu at (190.6, 57.9)
- added R17: R_20K, Resistor_SMD:R_0805_2012Metric, F.Cu at (216.0, 81.5)
- added R18: R_30K, Resistor_SMD:R_0805_2012Metric, F.Cu at (212.2, 81.5)
- added R19: R_7K, Resistor_SMD:R_0805_2012Metric, F.Cu at (194.0, 61.6)
- added R2: R_200, Resistor_SMD:R_0805_2012Metric, F.Cu at (167.1, 61.4)
- added R20: R, Resistor_SMD:R_0805_2012Metric, F.Cu at (197.5, 76.0)
- added R21: R, Resistor_SMD:R_0805_2012Metric, F.Cu at (200.4, 73.8)
- added R22: R, Resistor_SMD:R_0805_2012Metric, F.Cu at (201.4, 76.0)
- added R23: R_1K, Resistor_SMD:R_0805_2012Metric, F.Cu at (194.4, 84.4)
- added R24: R_3.2K, Resistor_SMD:R_0805_2012Metric, F.Cu at (197.6, 85.2)
- added R3: R_200, Resistor_SMD:R_0805_2012Metric, F.Cu at (162.8, 61.5)
- added R4: R_200, Resistor_SMD:R_0805_2012Metric, F.Cu at (158.7, 61.6)
- added R5: R_200, Resistor_SMD:R_0805_2012Metric, F.Cu at (154.6, 61.6)
- added R6: R_0, Resistor_SMD:R_0805_2012Metric, F.Cu at (159.3, 67.2)
- added R7: R_0, Resistor_SMD:R_0805_2012Metric, F.Cu at (155.2, 65.5)
- added R8: R_0, Resistor_SMD:R_0805_2012Metric, F.Cu at (151.0, 58.0)
- added R9: R_0, Resistor_SMD:R_0805_2012Metric, F.Cu at (151.0, 61.5)
- added RA1: 28 k, Resistor_SMD:R_0805_2012Metric, F.Cu at (176.4, 85.8)
- added RA2: 28 k, Resistor_SMD:R_0805_2012Metric, F.Cu at (180.6, 75.4)
- added RA3: 28 k, Resistor_SMD:R_0805_2012Metric, F.Cu at (153.9, 90.2)
- added RA4: 28 k, Resistor_SMD:R_0805_2012Metric, F.Cu at (179.6, 77.7)
- added RA5: 28 k, Resistor_SMD:R_0805_2012Metric, F.Cu at (140.2, 88.5)
- added RA6: 28 k, Resistor_SMD:R_0805_2012Metric, F.Cu at (179.9, 82.1)
- added RA7: 28 k, Resistor_SMD:R_0805_2012Metric, F.Cu at (136.7, 83.6)
- added RB1: 6.619k, Resistor_SMD:R_0805_2012Metric, F.Cu at (171.8, 87.5)
- added RB2: 13.518k, Resistor_SMD:R_0805_2012Metric, F.Cu at (185.1, 76.0)
- added RB3: 4.369k, Resistor_SMD:R_0805_2012Metric, F.Cu at (154.0, 93.9)
- added RB4: 10.522k, Resistor_SMD:R_0805_2012Metric, F.Cu at (183.8, 80.2)
- added RB5: 2.362k, Resistor_SMD:R_0805_2012Metric, F.Cu at (140.2, 92.1)
- added RB6: 7.844k, Resistor_SMD:R_0805_2012Metric, F.Cu at (176.9, 94.0)
- added RB7: 578, Resistor_SMD:R_0805_2012Metric, F.Cu at (133.8, 84.6)
- added U1: LM324, LM324:SOIC127P600X175-14N, F.Cu at (153.2, 75.6)
- added U11: LM555, LM555CM:SO08, F.Cu at (135.0, 92.0)
- added U13: LM555, LM555CM:SO08, F.Cu at (172.0, 93.9)
- added U14: STM32F072RBTx, Package_QFP:LQFP-64_10x10mm_P0.5mm, F.Cu at (170.2, 74.9)
- added U16: LM555, LM555CM:SO08, F.Cu at (128.8, 84.5)
- added U17: LM324, LM324:SOIC127P600X175-14N, F.Cu at (210.6, 74.4)
- added U2: LM324, LM324:SOIC127P600X175-14N, F.Cu at (142.6, 78.0)
- added U3: LM555, LM555CM:SO08, F.Cu at (160.7, 92.2)
- added U5: LM555, LM555CM:SO08, F.Cu at (189.9, 88.7)
- added U6: SN74HC02NSR, SN74HC02NSR:SN74HC02NSR, F.Cu at (186.7, 67.6)
- added U7: LM555, LM555CM:SO08, F.Cu at (148.5, 93.6)
- added U9: LM555, LM555CM:SO08, F.Cu at (182.5, 88.4)
- added Y1: Crystal_32MHz, FA-128_32.0000MF20X-K5:OSCCC200X160X50N, F.Cu at (161.2, 73.7)
- J1: value Conn_ARM_JTAG_SWD_10 -> Conn_01x07_Male; footprint Connector_PinHeader_1.27mm:PinHeader_2x05_P1.27mm_Vertical_SMD -> Connector_PinHeader_2.54mm:PinHeader_1x07_P2.54mm_Vertical
- Q1, Q2, Q3, Q4: value 2N3904 -> MMBT3904; footprint Package_TO_SOT_THT:TO-92_Inline -> Package_TO_SOT_SMD:SOT-23
- U4: value STM32F072RBTx -> U4; footprint Package_QFP:LQFP-64_10x10mm_P0.5mm -> NCP1117:NCP1117DT33T5G
- moved Q1 57.9 mm to (195.7, 69.4)
- moved Q3 57.4 mm to (200.5, 68.9)
- moved Q4 54.3 mm to (199.9, 61.7), turned to 90 degrees
- moved Q2 44.0 mm to (186.7, 59.1), turned to 270 degrees
- moved U4 38.0 mm to (143.9, 52.1), turned to 270 degrees
- moved J1 13.3 mm to (131.9, 75.8), turned to 180 degrees
Connections:
- J1 pad 1: Net-(J1-Pad1) -> /T7
- J1 pad 2: Net-(J1-Pad2) -> /T8
- J1 pad 3: Net-(J1-Pad3) -> /T9
- J1 pad 4: Net-(J1-Pad4) -> /T10
- J1 pad 5: Net-(J1-Pad3) -> /T11
- J1 pad 6: Net-(J1-Pad6) -> /T12
- J1 pad 7: Net-(J1-Pad7) -> /T13
- Q2 pad 2: Net-(Q2-Pad2) -> Net-(CR2-Pad2)
- Q3 pad 1: Net-(Q1-Pad3) -> Net-(Q3-Pad1)
- Q3 pad 2: Net-(Q3-Pad2) -> Net-(Q1-Pad3)
- Q4 pad 1: GND -> Net-(Q3-Pad1)
- Q4 pad 2: Net-(Q3-Pad2) -> GNDREF
- Q4 pad 3: Net-(Q2-Pad2) -> Net-(Q4-Pad3)
- U4 pad 1: Net-(U4-Pad1) -> GND
- U4 pad 2: Net-(U4-Pad2) -> +3V3
- U4 pad 3: Net-(U4-Pad3) -> VCC
Routing:
- net +3V3: track 0.00 -> 305.5 mm, vias 0 -> 9
- net VCC: track 0.00 -> 191.4 mm, vias 0 -> 9
- net +5V: track 0.00 -> 188.7 mm, vias 0 -> 13
- net GND: track 0.00 -> 151.7 mm, vias 0 -> 93
- net /T13: track 0.00 -> 138.1 mm, vias 0 -> 2
- net Net-(C1-Pad2): track 0.00 -> 120.4 mm, vias 0 -> 2
- net Net-(C2-Pad2): track 0.00 -> 99.3 mm, vias 0 -> 2
- net /D13: track 0.00 -> 97.5 mm, vias 0 -> 2
- net /D12: track 0.00 -> 96.8 mm, vias 0 -> 2
- net /D11: track 0.00 -> 93.6 mm, vias 0 -> 2
- net Net-(C5-Pad2): track 0.00 -> 80.1 mm
- net /ADSR_OUT: track 0.00 -> 74.3 mm, vias 0 -> 2
- net /T7: track 0.00 -> 66.3 mm, vias 0 -> 5
- net /SIGNAL: track 0.00 -> 59.9 mm, vias 0 -> 2
- net /D10: track 0.00 -> 59.8 mm, vias 0 -> 3
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- added copper zone on B.Cu, net GND
- added copper zone on F.Cu, net GND
Other:
- net class Default: trace_width 0.25 -> 0.1524; via_dia 0.8 -> 0.6096; via_drill 0.4 -> 0.3048
- rule trace_min: 0.2 -> 0.1524
- rule via_min_drill: 0.3 -> 0.3048
- rule via_min_size: 0.4 -> 0.6096
- board text added: "*"
