File: Synth - Final/new_synth_transistor.sch (KiCad schematic (older format))
At the start: 93 parts

Commit message: Add PCB
Parts:
- removed C? (x2): C_1nF, symbol Device:C
- removed C? (x2): C_22pF, symbol Device:C
- removed D?: D, symbol Device:D
- removed R? (x2): R_1M, symbol Device:R
- removed U? (x7): LMC6484, symbol Amplifier_Operational:LMC6484
- removed U? (x2): 7402, symbol 74xx:7402
- removed U?: LM324, SOIC127P600X175-14N, symbol LM324:LM324
- added C10, C7: C_22pF, Capacitor_SMD:C_0805_2012Metric, symbol Device:C
- added CR4: BAT60JFILM, BAT60JFILM:BAT60JFILM, symbol BAT60JFILM:BAT60JFILM
- added J7: UJ2-MIBH-4-SMT-TR, digikey-footprints:USB_Micro_B_Male_UJ2-MIBH-4-SMT-TR, symbol dk_USB-DVI-HDMI-Connectors:UJ2-MIBH-4-SMT-TR
- added R10, R23: R_1K, Resistor_SMD:R_0805_2012Metric, symbol Device:R
- added R11: R_4K, Resistor_SMD:R_0805_2012Metric, symbol Device:R
- added R24: R_3.2K, Resistor_SMD:R_0805_2012Metric, symbol Device:R
- added R8, R9: R_0, Resistor_SMD:R_0805_2012Metric, symbol Device:R
- added U1, U2: LM324, LM324:SOIC127P600X175-14N, symbol LM324:LM324
- added U6: SN74HC02NSR, SN74HC02NSR:SN74HC02NSR, symbol SN7402HC02NSR:SN74HC02NSR
- C1, C11, C12, C13, C14, C17, C2, C3, C4, C5, C6, C8, C9: renamed from C?; footprint (none) -> Capacitor_SMD:C_0805_2012Metric
- D1, D2, D3, D4, D5: renamed from D?; footprint (none) -> Diode_SMD:D_0805_2012Metric
- J1, J2, J3, J4: renamed from J?; footprint (none) -> Connector_PinHeader_2.54mm:PinHeader_1x07_P2.54mm_Vertical
- J5: renamed from J?; footprint (none) -> AU-Y1007:ASSMANN_AU-Y1007
- R1, R13, R16, R2, R3, R4, R5, R6, R7: renamed from R?; footprint (none) -> Resistor_SMD:R_0805_2012Metric
- R17: renamed from R?; value R_1K -> R_20K
- R18: renamed from R?; value R_2.2K -> R_30K
- R19: renamed from R?; value 10K -> R_7K
- RA1, RA2, RA3, RA4, RA5, RA6, RA7: renamed from RA?; footprint (none) -> Resistor_SMD:R_0805_2012Metric
- RB1, RB2, RB3, RB4, RB5, RB6, RB7: renamed from RB?; footprint (none) -> Resistor_SMD:R_0805_2012Metric
- U11, U13, U16, U3, U5, U7, U9: renamed from U?; footprint (none) -> LM555CM:SO08
- U17: renamed from U?; footprint SOIC127P600X175-14N -> LM324:SOIC127P600X175-14N
- Y1: renamed from Y?; footprint (none) -> FA-128_32.0000MF20X-K5:OSCCC200X160X50N
- gave numbers to parts that had none: 16
Connections:
- net +3V3: now also R6.1, R23.1, R8.1
- net GND: now also Y1.2, Y1.4, C10.2, C7.2, R24.2, R9.2, U1.11 (VCC-), U2.11 (VCC-), U6.7 (GND); no longer C17.2, Q4.2 (E), R13.2, R18.2, U17.11 (VCC-)
- net SIGNAL: now also U14.43 (PA10), U6.9 (3B)
- net T10: now also U1.1 (OUTPUT1), U1.2 (INVERTING_INPUT1)
- net T11: now also U2.6 (INVERTING_INPUT2), U2.7 (OUTPUT2)
- net T12: now also U1.13 (INVERTING_INPUT4), U1.14 (OUTPUT4)
- net T13: now also U2.1 (OUTPUT1), U2.2 (INVERTING_INPUT1)
- net T7: now also U2.13 (INVERTING_INPUT4), U2.14 (OUTPUT4)
- net T8: now also U1.8 (OUTPUT3), U1.9 (INVERTING_INPUT3)
- net T9: now also U1.6 (INVERTING_INPUT2), U1.7 (OUTPUT2)
- net VCC: now also R10.1, U1.4 (VCC+), U2.4 (VCC+), U6.14 (VCC); no longer R6.1, U17.6 (INVERTING_INPUT2)
- net at CR3.1, R13.1: now also U6.5 (2A)
- net 2B: now reaches R12.2, R19.2
- net 2B: now also U6.10 (3Y), U6.6 (2B)
- net at U14.5 (PF0), Y1.1: now also C7.1
- net at U14.6 (PF1), Y1.3: now also C10.1
- net at C2.2, RB2.1, U5.2 (TR)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: now also U2.3 (NON-INVERTING_INPUT1)
- net at C4.2, RB4.1, U9.2 (TR)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: now also U1.12 (NON-INVERTING_INPUT4)
- net at C12.2, RB6.1, U13.2 (TR)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: now also U2.5 (NON-INVERTING_INPUT2)
- net at C14.2, RB7.1, U16.2 (TR)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: now also U2.12 (NON-INVERTING_INPUT4)
- net at C1.2, RB1.1, U3.2 (TR)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: now also U1.3 (NON-INVERTING_INPUT1)
- net 3A: now reaches CR1.2, CR2.1
- net 3A: now also U6.4 (2Y), U6.8 (3A)
- net at U17.8 (OUTPUT3), U17.9 (INVERTING_INPUT3): now also CR4.1
- net at Q1.2 (E): now also CR4.2
- net at C3.2, RB3.1, U7.2 (TR)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: now also U1.5 (NON-INVERTING_INPUT2)
- net at C5.2, RB5.1, U11.2 (TR)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: now also U1.10 (NON-INVERTING_INPUT3)
- net Reset: no longer names the net of U14.7 (NRST)
- net Reset: now also R8.2, R9.1; no longer J6.10 (~RESET~)
- new net: R10.2, R11.1, U17.6 (INVERTING_INPUT2)
- new net GNDREF: C17.2, Q4.2 (E), R11.2, R13.2, R18.2, R23.2, R24.1, U17.11 (VCC-)
- no-connect marks 39 -> 45
Other:
- note added: "DO WE USE GNDREF or GND for powering op-amp\n"
- note added: "Virtual Ground"
- moved on the sheet: R6, R7, Y1
