File: Synth - Final/_saved_new_synth_transistor.sch (KiCad schematic (older format))
At the start: 88 parts, among them J1 Conn_01x07_Male, J2 Conn_01x07_Male, J3 Conn_01x07_Male, J4 Conn_01x07_Male, J5 USB_B, J6 Conn_ARM_JTAG_SWD_10, Q1 MMBT3904, Q2 MMBT3904, Q3 MMBT3904, Q4 MMBT3904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

Commit message: Update pcb layout
Parts:
- gave numbers to parts that had none: 2
Changed lines of the file:
@@
 	16300 2600 16650 2600
 $Comp
-L power:+3.3V #PWR?
+L power:+3.3V #PWR014
 U 1 1 5DF8F455
 P 9050 7700
-F 0 "#PWR?" H 9050 7550 50  0001 C CNN
+F 0 "#PWR014" H 9050 7550 50  0001 C CNN
 F 1 "+3.3V" H 9065 7873 50  0000 C CNN
 F 2 "" H 9050 7700 50  0001 C CNN
@@
 $EndComp
 $Comp
-L power:+3.3V #PWR?
+L power:+3.3V #PWR015
 U 1 1 5DF8F533
 P 9550 7100
-F 0 "#PWR?" H 9550 6950 50  0001 C CNN
+F 0 "#PWR015" H 9550 6950 50  0001 C CNN
 F 1 "+3.3V" H 9565 7273 50  0000 C CNN
 F 2 "" H 9550 7100 50  0001 C CNN
@@
 $EndComp
 $Comp
-L Connector:USB_B J?
+L Connector:USB_B J7
 U 1 1 5DCCF9F3
 P 14350 9800
-F 0 "J?" H 14405 10267 50  0000 C CNN
+F 0 "J7" H 14405 10267 50  0000 C CNN
 F 1 "USB_B" H 14405 10176 50  0000 C CNN
 F 2 "AU-Y1007:ASSMANN_AU-Y1007" H 14500 9750 50  0001 C CNN
@@
 NoConn ~ 14650 9900
 $Comp
-L power:+5VD #PWR?
+L power:+5VD #PWR017
 U 1 1 5DD1B176
 P 14750 9600
-F 0 "#PWR?" H 14750 9450 50  0001 C CNN
+F 0 "#PWR017" H 14750 9450 50  0001 C CNN
 F 1 "+5VD" H 14765 9773 50  0000 C CNN
 F 2 "" H 14750 9600 50  0001 C CNN
@@
 $EndComp
 $Comp
-L power:Earth #PWR?
+L power:Earth #PWR016
 U 1 1 5DD1B2BD
 P 14300 10250
-F 0 "#PWR?" H 14300 10000 50  0001 C CNN
+F 0 "#PWR016" H 14300 10000 50  0001 C CNN
 F 1 "Earth" H 14300 10100 50  0001 C CNN
 F 2 "" H 14300 10250 50  0001 C CNN
@@
 $EndComp
 $Comp
-L Connector:Conn_01x02_Male J?
+L Connector:Conn_01x02_Male J8
 U 1 1 5DD1B3D3
 P 15450 9950
-F 0 "J?" H 15556 10128 50  0000 C CNN
+F 0 "J8" H 15556 10128 50  0000 C CNN
 F 1 "Conn_01x02_Male" H 15556 10037 50  0000 C CNN
 F 2 "Connector_PinHeader_2.54mm:PinHeader_1x02_P2.54mm_Vertical" H 15450 9950 50  0001 C CNN
@@
 	16050 9950 16050 9850
 $Comp
-L power:+5VD #PWR?
+L power:+5VD #PWR019
 U 1 1 5DD3556C
 P 16050 9850
-F 0 "#PWR?" H 16050 9700 50  0001 C CNN
+F 0 "#PWR019" H 16050 9700 50  0001 C CNN
 F 1 "+5VD" H 16065 10023 50  0000 C CNN
 F 2 "" H 16050 9850 50  0001 C CNN
@@
 $EndComp
 $Comp
-L power:Earth #PWR?
+L power:Earth #PWR018
 U 1 1 5DD3566F
 P 15650 10050
-F 0 "#PWR?" H 15650 9800 50  0001 C CNN
+F 0 "#PWR018" H 15650 9800 50  0001 C CNN
 F 1 "Earth" H 15650 9900 50  0001 C CNN
 F 2 "" H 15650 10050 50  0001 C CNN
