File: Teensy - Synth/new_synth_transistor.sch (KiCad schematic (older format))
At the start: 58 parts, among them J1 Conn_01x07_Female, Q1 MMBT3904, Q2 MMBT3904, Q3 MMBT3904, Q4 MMBT3904, U1 LM324, U11 LM555, U13 LM555, U16 LM555, U17 LM324, U2 LM324, U3 LM555, U4 Teensy3.6, U5 LM555, U6 SN74HC02NSR, U7 LM555, U9 LM555

Commit message: Revert to Teesy PCB files
Parts:
- U1, U17, U2: symbol new_synth_transistor-rescue:LM324-LM324 -> LM324:LM324
- renumbered J1 to J?, U4 to U?
Changed lines of the file:
@@
 	18900 2200 18900 2350
 $Comp
-L new_synth_transistor-rescue:LM324-LM324 U17
+L LM324:LM324 U17
 U 1 1 5DC5D391
 P 21800 3600
@@
 $EndComp
 $Comp
-L new_synth_transistor-rescue:LM324-LM324 U17
+L LM324:LM324 U17
 U 2 1 5DC68A05
 P 21850 2600
@@
 $EndComp
 $Comp
-L new_synth_transistor-rescue:LM324-LM324 U17
+L LM324:LM324 U17
 U 3 1 5DC68B40
 P 19500 4900
@@
 Connection ~ 20150 4000
 $Comp
-L new_synth_transistor-rescue:LM324-LM324 U2
+L LM324:LM324 U2
 U 1 1 5DEEF739
 P 2650 1400
@@
 $EndComp
 $Comp
-L new_synth_transistor-rescue:LM324-LM324 U2
+L LM324:LM324 U2
 U 2 1 5DEEF88A
 P 10750 1450
@@
 $EndComp
 $Comp
-L new_synth_transistor-rescue:LM324-LM324 U1
+L LM324:LM324 U1
 U 3 1 5DEEF97F
 P 8450 4200
@@
 $EndComp
 $Comp
-L new_synth_transistor-rescue:LM324-LM324 U2
+L LM324:LM324 U2
 U 4 1 5DEF0107
 P 12600 4300
@@
 Connection ~ 12900 4400
 $Comp
-L new_synth_transistor-rescue:LM324-LM324 U1
+L LM324:LM324 U1
 U 1 1 5DFC22FC
 P 1550 4400
@@
 $EndComp
 $Comp
-L new_synth_transistor-rescue:LM324-LM324 U1
+L LM324:LM324 U1
 U 2 1 5DFC2465
 P 4850 4400
@@
 Connection ~ 11050 1550
 $Comp
-L new_synth_transistor-rescue:LM324-LM324 U1
+L LM324:LM324 U1
 U 4 1 5E208FFB
 P 6600 1450
@@
 	16300 2600 16650 2600
 $Comp
-L new_synth_transistor-rescue:Teensy3.6-teensy U4
+L new_synth_transistor-rescue:Teensy3.6-teensy U?
 U 1 1 5DDCBF53
 P 11350 8500
-F 0 "U4" H 11350 11043 60  0000 C CNN
+F 0 "U?" H 11350 11043 60  0000 C CNN
 F 1 "Teensy3.6" H 11350 10937 60  0000 C CNN
 F 2 "teensy:Teensy35_36" H 11350 10831 60  0000 C CNN
@@
 $EndComp
 $Comp
-L power:GND #PWR0101
+L power:GND #PWR?
 U 1 1 5DDEB10D
 P 9800 6350
-F 0 "#PWR0101" H 9800 6100 50  0001 C CNN
+F 0 "#PWR?" H 9800 6100 50  0001 C CNN
 F 1 "GND" H 9805 6177 50  0000 C CNN
 F 2 "" H 9800 6350 50  0001 C CNN
@@
 $EndComp
 $Comp
-L power:GND #PWR0103
+L power:GND #PWR?
 U 1 1 5DDEB3CC
 P 9750 9000
-F 0 "#PWR0103" H 9750 8750 50  0001 C CNN
+F 0 "#PWR?" H 9750 8750 50  0001 C CNN
 F 1 "GND" H 9755 8827 50  0000 C CNN
 F 2 "" H 9750 9000 50  0001 C CNN
@@
 $EndComp
 $Comp
-L power:GND #PWR0104
+L power:GND #PWR?
 U 1 1 5DE16CCF
 P 9750 10150
-F 0 "#PWR0104" H 9750 9900 50  0001 C CNN
+F 0 "#PWR?" H 9750 9900 50  0001 C CNN
 F 1 "GND" H 9755 9977 50  0000 C CNN
 F 2 "" H 9750 10150 50  0001 C CNN
@@
 $EndComp
 $Comp
-L power:GNDREF #PWR0105
+L power:GNDREF #PWR?
 U 1 1 5DE9A32C
 P 17650 2950
-F 0 "#PWR0105" H 17650 2700 50  0001 C CNN
+F 0 "#PWR?" H 17650 2700 50  0001 C CNN
 F 1 "GNDREF" H 17655 2777 50  0000 C CNN
 F 2 "" H 17650 2950 50  0001 C CNN
@@
 $EndComp
 $Comp
-L power:GND #PWR0107
+L power:GND #PWR?
 U 1 1 5DEBC158
 P 13450 9950
-F 0 "#PWR0107" H 13450 9700 50  0001 C CNN
+F 0 "#PWR?" H 13450 9700 50  0001 C CNN
 F 1 "GND" H 13455 9777 50  0000 C CNN
 F 2 "" H 13450 9950 50  0001 C CNN
@@
 $EndComp
 $Comp
-L power:VCC #PWR0108
+L power:VCC #PWR?
 U 1 1 5DF08F0C
 P 12850 9600
-F 0 "#PWR0108" H 12850 9450 50  0001 C CNN
+F 0 "#PWR?" H 12850 9450 50  0001 C CNN
 F 1 "VCC" H 12867 9773 50  0000 C CNN
 F 2 "" H 12850 9600 50  0001 C CNN
@@
 	12850 9850 12500 9850
 $Comp
-L power:+3V3 #PWR0110
+L power:+3V3 #PWR?
 U 1 1 5DF396E1
 P 13150 9600
-F 0 "#PWR0110" H 13150 9450 50  0001 C CNN
+F 0 "#PWR?" H 13150 9450 50  0001 C CNN
 F 1 "+3V3" H 13165 9773 50  0000 C CNN
 F 2 "" H 13150 9600 50  0001 C CNN
@@
 $EndComp
 $Comp
-L power:+3V3 #PWR0111
+L power:+3V3 #PWR?
 U 1 1 5DF399B2
 P 9750 8850
-F 0 "#PWR0111" H 9750 8700 50  0001 C CNN
+F 0 "#PWR?" H 9750 8700 50  0001 C CNN
 F 1 "+3V3" H 9765 9023 50  0000 C CNN
 F 2 "" H 9750 8850 50  0001 C CNN
@@
 	10200 8850 9750 8850
 $Comp
-L power:+3V3 #PWR0112
+L power:+3V3 #PWR?
 U 1 1 5DF4A1C6
 P 9750 7750
-F 0 "#PWR0112" H 9750 7600 50  0001 C CNN
+F 0 "#PWR?" H 9750 7600 50  0001 C CNN
 F 1 "+3V3" H 9765 7923 50  0000 C CNN
 F 2 "" H 9750 7750 50  0001 C CNN
@@
 	12850 9850 12850 9600
 $Comp
-L power:VCC #PWR0114
+L power:VCC #PWR?
 U 1 1 5DF20964
 P 12600 5150
-F 0 "#PWR0114" H 12600 5000 50  0001 C CNN
+F 0 "#PWR?" H 12600 5000 50  0001 C CNN
 F 1 "VCC" H 12617 5323 50  0000 C CNN
 F 2 "" H 12600 5150 50  0001 C CNN
@@
 	12900 5150 12600 5150
 $Comp
-L power:VCC #PWR0136
+L power:VCC #PWR?
 U 1 1 5DF30D58
 P 10750 2300
-F 0 "#PWR0136" H 10750 2150 50  0001 C CNN
+F 0 "#PWR?" H 10750 2150 50  0001 C CNN
 F 1 "VCC" H 10767 2473 50  0000 C CNN
 F 2 "" H 10750 2300 50  0001 C CNN
@@
 	11050 2300 10750 2300
 $Comp
-L power:VCC #PWR0137
+L power:VCC #PWR?
 U 1 1 5DF510AB
 P 8450 5100
-F 0 "#PWR0137" H 8450 4950 50  0001 C CNN
+F 0 "#PWR?" H 8450 4950 50  0001 C CNN
 F 1 "VCC" H 8467 5273 50  0000 C CNN
 F 2 "" H 8450 5100 50  0001 C CNN
@@
 	8750 5100 8450 5100
 $Comp
-L power:VCC #PWR0138
+L power:VCC #PWR?
 U 1 1 5DF63217
 P 6600 2300
-F 0 "#PWR0138" H 6600 2150 50  0001 C CNN
+F 0 "#PWR?" H 6600 2150 50  0001 C CNN
 F 1 "VCC" H 6617 2473 50  0000 C CNN
 F 2 "" H 6600 2300 50  0001 C CNN
@@
 	6900 2300 6600 2300
 $Comp
-L power:VCC #PWR0139
+L power:VCC #PWR?
 U 1 1 5DF73926
 P 4850 5250
-F 0 "#PWR0139" H 4850 5100 50  0001 C CNN
+F 0 "#PWR?" H 4850 5100 50  0001 C CNN
 F 1 "VCC" H 4867 5423 50  0000 C CNN
 F 2 "" H 4850 5250 50  0001 C CNN
@@
 	5150 5250 4850 5250
 $Comp
-L power:VCC #PWR0140
+L power:VCC #PWR?
 U 1 1 5DF842FC
 P 1550 5250
-F 0 "#PWR0140" H 1550 5100 50  0001 C CNN
+F 0 "#PWR?" H 1550 5100 50  0001 C CNN
 F 1 "VCC" H 1567 5423 50  0000 C CNN
 F 2 "" H 1550 5250 50  0001 C CNN
@@
 	1850 5250 1550 5250
 $Comp
-L power:VCC #PWR0141
+L power:VCC #PWR?
 U 1 1 5DF94FE1
 P 2650 2250
-F 0 "#PWR0141" H 2650 2100 50  0001 C CNN
+F 0 "#PWR?" H 2650 2100 50  0001 C CNN
 F 1 "VCC" H 2667 2423 50  0000 C CNN
 F 2 "" H 2650 2250 50  0001 C CNN
@@
 	2950 2250 2650 2250
 $Comp
-L power:VCC #PWR0142
+L power:VCC #PWR?
 U 1 1 5DFA7AE0
 P 8600 10700
-F 0 "#PWR0142" H 8600 10550 50  0001 C CNN
+F 0 "#PWR?" H 8600 10550 50  0001 C CNN
 F 1 "VCC" H 8618 10873 50  0000 C CNN
 F 2 "" H 8600 10700 50  0001 C CNN
@@
 $EndComp
 $Comp
-L power:+5V #PWR0143
+L power:+5V #PWR?
 U 1 1 5DFA7B90
 P 8600 10700
-F 0 "#PWR0143" H 8600 10550 50  0001 C CNN
+F 0 "#PWR?" H 8600 10550 50  0001 C CNN
 F 1 "+5V" H 8615 10873 50  0000 C CNN
 F 2 "" H 8600 10700 50  0001 C CNN
@@
 NoConn ~ 12500 9750
 $Comp
-L Connector:Conn_01x07_Female J1
+L Connector:Conn_01x07_Female J?
 U 1 1 5E203275
 P 7850 9450
-F 0 "J1" H 7877 9476 50  0000 L CNN
+F 0 "J?" H 7877 9476 50  0000 L CNN
 F 1 "Conn_01x07_Female" H 7877 9385 50  0000 L CNN
 F 2 "" H 7850 9450 50  0001 C CNN

Commit message: Adding new paths for libraries, new component annotations, and netlist
Parts:
- removed U?: Teensy3.6, teensy:Teensy35_36, symbol new_synth_transistor-rescue:Teensy3.6-teensy
- added U8: Teensy3.6, teensy:Teensy35_36, symbol teensy:Teensy3.6
- gave numbers to parts that had none: 1
- renumbered C12 to C6, C14 to C7, C17 to C8, CR4 to CR2, CR2 to CR3, CR3 to CR4, R23 to R1, R19 to R10, R20 to R11, R21 to R12, R22 to R13, R10 to R14, R11 to R15, R24 to R2, R12 to R3, R13 to R4, R14 to R5, R15 to R6, R16 to R7, R17 to R8, R18 to R9, U16 to U10, U6 to U11, U17 to U12, U17 to U2, U5 to U4, U7 to U5, U9 to U6, U11 to U7, U13 to U9
Connections:
- net +3V3: now also U8.15 (3.3V), U8.26 (3V3), U8.51 (3.3V)
- net +5V: now also U8.53 (VIN)
- net GND: now also U8.1 (GND), U8.27 (GND), U8.39 (GND), U8.52 (AGND), U8.55 (AREF)
- net L1: now also U8.30 (33_A14_CAN1TX_SCL0)
- net L2: now also U8.31 (34_A15_CAN1TX_SDA0)
- net L3: now also U8.32 (35_A16_PWM)
- net L4: now also U8.33 (36_A17_PWM)
- net L5: now also U8.34 (37_A18_PWM_SCL1)
- net L6: now also U8.35 (38_A19_PWM_SDA1)
- net L7: now also U8.36 (39_A20)
- net T1: now also U8.50 (23_A9_PWM_TOUCH)
- net T2: now also U8.49 (22_A8_PWM_TOUCH)
- net T3: now also U8.48 (21_A7_PWM_CS0_SCK1)
- net T4: now also U8.47 (20_A6_PWM_CS0_SCK1)
- net T5: now also U8.46 (19_A5_SCL0_TOUCH)
- net T6: now also U8.45 (18_A4_SDA0_TOUCH)
- net T7: now also U8.44 (17_A3_SDA0_TOUCH)
- net TONE: now also U8.38 (A22_DAC1)
