File: Teensy - Synth/new_synth_transistor.sch (KiCad schematic (older format))
At the start: 58 parts, among them J1 Conn_01x07_Female, Q1 MMBT3904, Q2 MMBT3904, Q3 MMBT3904, Q4 MMBT3904, U1 LM324, U10 LM555, U11 SN74HC02NSR, U12 LM324, U2 LM324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

Commit message: website gallery formatting and libraries and layout (almost done)
Parts:
- added unit 3 of U2
- U8: symbol teensy:Teensy3.6 -> new_synth_transistor-rescue:Teensy3.6-teensy
- renumbered U2 to U12
Connections:
- no-connect marks 50 -> 53
Changed lines of the file:
@@
 $EndComp
 $Comp
-L LM324:LM324 U2
+L LM324:LM324 U12
 U 3 1 5DC68B40
 P 19500 4900
-F 0 "U2" H 19500 5270 50  0000 C CNN
+F 0 "U12" H 19500 5270 50  0000 C CNN
 F 1 "LM324" H 19500 5179 50  0000 C CNN
 F 2 "LM324:SOIC127P600X175-14N" H 19500 4900 50  0001 L BNN
@@
 	-1   0    0    -1
 $EndComp
-Connection ~ 19200 4900
 $Comp
 L power:VCC #PWR055
@@
 F 1 "LM324" H 2650 950 50  0000 C CNN
 F 2 "LM324:SOIC127P600X175-14N" H 2650 1400 50  0001 L BNN
-F 3 "these devices consist of four independent high-gain frequency-compensated operational amplifiers that are designed sp..." H 2650 1400 50  0001 L BNN
+F 3 "" H 2650 1400 50  0001 L BNN
 F 4 "Texas Instruments" H 2650 1400 50  0001 L BNN "Field4"
 F 5 "Unavailable" H 2650 1400 50  0001 L BNN "Field5"
@@
 F 1 "LM324" H 10750 1100 50  0000 C CNN
 F 2 "LM324:SOIC127P600X175-14N" H 10750 1450 50  0001 L BNN
-F 3 "these devices consist of four independent high-gain frequency-compensated operational amplifiers that are designed sp..." H 10750 1450 50  0001 L BNN
+F 3 "" H 10750 1450 50  0001 L BNN
 F 4 "Texas Instruments" H 10750 1450 50  0001 L BNN "Field4"
 F 5 "Unavailable" H 10750 1450 50  0001 L BNN "Field5"
@@
 F 1 "LM324" H 12600 3950 50  0000 C CNN
 F 2 "LM324:SOIC127P600X175-14N" H 12600 4300 50  0001 L BNN
-F 3 "these devices consist of four independent high-gain frequency-compensated operational amplifiers that are designed sp..." H 12600 4300 50  0001 L BNN
+F 3 "" H 12600 4300 50  0001 L BNN
 F 4 "Texas Instruments" H 12600 4300 50  0001 L BNN "Field4"
 F 5 "Unavailable" H 12600 4300 50  0001 L BNN "Field5"
@@
 	-1   0    0    1
 $EndComp
-Connection ~ 12300 4300
-Connection ~ 12900 4400
 $Comp
 L LM324:LM324 U1
@@
 	-1   0    0    1
 $EndComp
-Connection ~ 4550 4400
-Connection ~ 5150 4500
-Connection ~ 8150 4200
-Connection ~ 8750 4300
-Connection ~ 10450 1450
-Connection ~ 11050 1550
 $Comp
 L LM324:LM324 U1
@@
 	-1   0    0    1
 $EndComp
-Connection ~ 6300 1450
-Connection ~ 6900 1550
 $Comp
 L power:VCC #PWR06
@@
 Wire Wire Line
 	1350 4700 1550 4700
-Connection ~ 1850 4500
 Wire Wire Line
 	1850 4050 1150 4050
@@
 Wire Wire Line
 	1150 4400 1250 4400
-Connection ~ 2350 1400
-Connection ~ 2950 1500
 Wire Wire Line
 	2350 1050 2950 1050
@@
 TONE
 $Comp
-L teensy:Teensy3.6 U8
+L new_synth_transistor-rescue:Teensy3.6-teensy U8
 U 1 1 5DDD7864
 P 11350 8500
@@
 	1    0    0    -1
 $EndComp
+$Comp
+L LM324:LM324 U2
+U 3 1 5DE30E7F
+P 21600 5200
+F 0 "U2" H 21600 5570 50  0000 C CNN
+F 1 "LM324" H 21600 5479 50  0000 C CNN
+F 2 "LM324:SOIC127P600X175-14N" H 21600 5200 50  0001 L BNN
+F 3 "" H 21600 5200 50  0001 L BNN
+F 4 "Texas Instruments" H 21600 5200 50  0001 L BNN "Field4"
+F 5 "Unavailable" H 21600 5200 50  0001 L BNN "Field5"
+F 6 "None" H 21600 5200 50  0001 L BNN "Field6"
+F 7 "LM324" H 21600 5200 50  0001 L BNN "Field7"
+F 8 "SOIC-14 Texas Instruments" H 21600 5200 50  0001 L BNN "Field8"
+	3    21600 5200
+	-1   0    0    -1
+$EndComp
+NoConn ~ 21300 5200
+NoConn ~ 21900 5100
+NoConn ~ 21900 5300
 $EndSCHEMATC

Commit message: final layout, no dxf
Connections:
- net T1: now also U1.13 (INVERTING_INPUT4), U1.14 (OUTPUT4); no longer U2.13 (INVERTING_INPUT4), U2.14 (OUTPUT4)
- net T2: now also U1.8 (OUTPUT3), U1.9 (INVERTING_INPUT3); no longer U2.6 (INVERTING_INPUT2), U2.7 (OUTPUT2)
- net T3: now also U1.6 (INVERTING_INPUT2), U1.7 (OUTPUT2); no longer U1.8 (OUTPUT3), U1.9 (INVERTING_INPUT3)
- net T4: now also U1.1 (OUTPUT1), U1.2 (INVERTING_INPUT1); no longer U1.13 (INVERTING_INPUT4), U1.14 (OUTPUT4)
- net T5: now also U2.6 (INVERTING_INPUT2), U2.7 (OUTPUT2); no longer U1.6 (INVERTING_INPUT2), U1.7 (OUTPUT2)
- net T7: now also U2.13 (INVERTING_INPUT4), U2.14 (OUTPUT4); no longer U1.1 (OUTPUT1), U1.2 (INVERTING_INPUT1)
Other:
- moved on the sheet: U2C
Changed lines of the file:
@@
 T6
 Text Label 1100 4400 2    50   ~ 0
-T7
+T4
 Text Label 4500 4400 2    50   ~ 0
-T5
+T3
 Wire Wire Line
 	4500 4400 4550 4400
 Text Label 8100 4200 2    50   ~ 0
-T3
+T2
 Wire Wire Line
 	8100 4200 8150 4200
 Text Label 12250 4300 2    50   ~ 0
-T1
+T7
 Wire Wire Line
 	12250 4300 12300 4300
 Text Label 10400 1450 2    50   ~ 0
-T2
+T5
 Wire Wire Line
 	10400 1450 10450 1450
 Text Label 6250 1450 2    50   ~ 0
-T4
+T1
 Wire Wire Line
 	6250 1450 6300 1450
@@
 	20150 4000 19900 4000
 Connection ~ 20150 4000
-$Comp
-L LM324:LM324 U2
-U 1 1 5DEEF739
-P 2650 1400
-F 0 "U2" H 2650 850 50  0000 C CNN
-F 1 "LM324" H 2650 950 50  0000 C CNN
-F 2 "LM324:SOIC127P600X175-14N" H 2650 1400 50  0001 L BNN
-F 3 "" H 2650 1400 50  0001 L BNN
-F 4 "Texas Instruments" H 2650 1400 50  0001 L BNN "Field4"
-F 5 "Unavailable" H 2650 1400 50  0001 L BNN "Field5"
-F 6 "None" H 2650 1400 50  0001 L BNN "Field6"
-F 7 "LM324" H 2650 1400 50  0001 L BNN "Field7"
-F 8 "SOIC-14 Texas Instruments" H 2650 1400 50  0001 L BNN "Field8"
-	1    2650 1400
-	-1   0    0    1
-$EndComp
 $Comp
 L LM324:LM324 U2
@@
 	1    0    0    -1
 $EndComp
+NoConn ~ 2350 2950
+NoConn ~ 2950 2850
+NoConn ~ 2950 3050
+$Comp
+L LM324:LM324 U2
+U 1 1 5DEEF739
+P 2650 1400
+F 0 "U2" H 2650 850 50  0000 C CNN
+F 1 "LM324" H 2650 950 50  0000 C CNN
+F 2 "LM324:SOIC127P600X175-14N" H 2650 1400 50  0001 L BNN
+F 3 "" H 2650 1400 50  0001 L BNN
+F 4 "Texas Instruments" H 2650 1400 50  0001 L BNN "Field4"
+F 5 "Unavailable" H 2650 1400 50  0001 L BNN "Field5"
+F 6 "None" H 2650 1400 50  0001 L BNN "Field6"
+F 7 "LM324" H 2650 1400 50  0001 L BNN "Field7"
+F 8 "SOIC-14 Texas Instruments" H 2650 1400 50  0001 L BNN "Field8"
+	1    2650 1400
+	-1   0    0    1
+$EndComp
 $Comp
 L LM324:LM324 U2
 U 3 1 5DE30E7F
-P 21600 5200
-F 0 "U2" H 21600 5570 50  0000 C CNN
-F 1 "LM324" H 21600 5479 50  0000 C CNN
-F 2 "LM324:SOIC127P600X175-14N" H 21600 5200 50  0001 L BNN
-F 3 "" H 21600 5200 50  0001 L BNN
-F 4 "Texas Instruments" H 21600 5200 50  0001 L BNN "Field4"
-F 5 "Unavailable" H 21600 5200 50  0001 L BNN "Field5"
-F 6 "None" H 21600 5200 50  0001 L BNN "Field6"
-F 7 "LM324" H 21600 5200 50  0001 L BNN "Field7"
-F 8 "SOIC-14 Texas Instruments" H 21600 5200 50  0001 L BNN "Field8"
-	3    21600 5200
+P 2650 2950
+F 0 "U2" H 2650 3320 50  0000 C CNN
+F 1 "LM324" H 2650 3229 50  0000 C CNN
+F 2 "LM324:SOIC127P600X175-14N" H 2650 2950 50  0001 L BNN
+F 3 "" H 2650 2950 50  0001 L BNN
+F 4 "Texas Instruments" H 2650 2950 50  0001 L BNN "Field4"
+F 5 "Unavailable" H 2650 2950 50  0001 L BNN "Field5"
+F 6 "None" H 2650 2950 50  0001 L BNN "Field6"
+F 7 "LM324" H 2650 2950 50  0001 L BNN "Field7"
+F 8 "SOIC-14 Texas Instruments" H 2650 2950 50  0001 L BNN "Field8"
+	3    2650 2950
 	-1   0    0    -1
 $EndComp
-NoConn ~ 21300 5200
-NoConn ~ 21900 5100
-NoConn ~ 21900 5300
 $EndSCHEMATC

Commit message: Add ADSR Signal
Parts:
- U1, U12, U2: symbol LM324:LM324 -> new_synth_transistor-rescue:LM324-LM324
Connections:
- net ADSR_OUT: now also U8.41 (14_A0_PWM_SCK0)
- net SIGNAL: now also U8.37 (A21_DAC0)
Changed lines of the file:
@@
 	18900 2200 18900 2350
 $Comp
-L LM324:LM324 U12
+L new_synth_transistor-rescue:LM324-LM324 U12
 U 1 1 5DC5D391
 P 21800 3600
@@
 $EndComp
 $Comp
-L LM324:LM324 U12
+L new_synth_transistor-rescue:LM324-LM324 U12
 U 2 1 5DC68A05
 P 21850 2600
@@
 $EndComp
 $Comp
-L LM324:LM324 U12
+L new_synth_transistor-rescue:LM324-LM324 U12
 U 3 1 5DC68B40
 P 19500 4900
@@
 Connection ~ 20150 4000
 $Comp
-L LM324:LM324 U2
+L new_synth_transistor-rescue:LM324-LM324 U2
 U 2 1 5DEEF88A
 P 10750 1450
@@
 $EndComp
 $Comp
-L LM324:LM324 U1
+L new_synth_transistor-rescue:LM324-LM324 U1
 U 3 1 5DEEF97F
 P 8450 4200
@@
 $EndComp
 $Comp
-L LM324:LM324 U2
+L new_synth_transistor-rescue:LM324-LM324 U2
 U 4 1 5DEF0107
 P 12600 4300
@@
 $EndComp
 $Comp
-L LM324:LM324 U1
+L new_synth_transistor-rescue:LM324-LM324 U1
 U 1 1 5DFC22FC
 P 1550 4400
@@
 $EndComp
 $Comp
-L LM324:LM324 U1
+L new_synth_transistor-rescue:LM324-LM324 U1
 U 2 1 5DFC2465
 P 4850 4400
@@
 $EndComp
 $Comp
-L LM324:LM324 U1
+L new_synth_transistor-rescue:LM324-LM324 U1
 U 4 1 5E208FFB
 P 6600 1450
@@
 L power:GND #PWR028
 U 1 1 5DE16CCF
-P 9750 10150
-F 0 "#PWR028" H 9750 9900 50  0001 C CNN
-F 1 "GND" H 9755 9977 50  0000 C CNN
-F 2 "" H 9750 10150 50  0001 C CNN
-F 3 "" H 9750 10150 50  0001 C CNN
-	1    9750 10150
+P 9650 10150
+F 0 "#PWR028" H 9650 9900 50  0001 C CNN
+F 1 "GND" H 9655 9977 50  0000 C CNN
+F 2 "" H 9650 10150 50  0001 C CNN
+F 3 "" H 9650 10150 50  0001 C CNN
+	1    9650 10150
 	1    0    0    -1
 $EndComp
@@
 Wire Wire Line
 	10200 6350 9800 6350
-Wire Wire Line
-	10200 10150 9750 10150
 Connection ~ 17650 2350
 $Comp
@@
 NoConn ~ 2950 3050
 $Comp
-L LM324:LM324 U2
+L new_synth_transistor-rescue:LM324-LM324 U2
 U 1 1 5DEEF739
 P 2650 1400
@@
 $EndComp
 $Comp
-L LM324:LM324 U2
+L new_synth_transistor-rescue:LM324-LM324 U2
 U 3 1 5DE30E7F
 P 2650 2950
@@
 	-1   0    0    -1
 $EndComp
+Text Label 10200 10350 2    50   ~ 0
+ADSR_OUT
+Wire Wire Line
+	9650 10150 10200 10150
+Text Label 10200 9950 2    50   ~ 0
+SIGNAL
 $EndSCHEMATC
