File: Teensy - Synth/new_synth_transistor.kicad_pcb (KiCad board)
At the start: 2 copper layers, 72.1 x 109.8 mm, 58 parts, among them J1 Conn_01x07_Female, Q1 MMBT3904, Q2 MMBT3904, Q3 MMBT3904, Q4 MMBT3904, U1 LM324, U10 LM555, U11 SN74HC02NSR, U12 LM324, U2 LM324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

Commit message: Updates to PCB
Routing:
- net (no net): track 31.4 -> 7.62 mm, vias 1 -> 0
- net GND: track 105.9 -> 114.6 mm, vias 23 -> 25
Changed lines of the file:
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@@
-(kicad_pcb (version 20171130) (host pcbnew 5.0.1-33cea8e~68~ubuntu18.04.1)
+(kicad_pcb (version 20171130) (host pcbnew "(5.0.1)-4")
   (general
     (thickness 1.6)
     (drawings 8)
-    (tracks 551)
+    (tracks 555)
     (zones 0)
     (modules 58)
@@
   (segment (start 269.651529 39.753212) (end 270.921529 39.753212) (width 0.1524) (layer F.Cu) (net 0))
   (segment (start 272.191529 39.753212) (end 270.921529 39.753212) (width 0.1524) (layer F.Cu) (net 0))
-  (segment (start 272.191529 39.753212) (end 272.191529 43.365713) (width 0.1524) (layer F.Cu) (net 0))
-  (segment (start 272.191529 43.365713) (end 272.18982 43.367422) (width 0.1524) (layer F.Cu) (net 0))
-  (segment (start 271.44472 44.112522) (end 271.44472 63.25896) (width 0.1524) (layer GND) (net 0))
-  (segment (start 272.18982 43.367422) (end 271.44472 44.112522) (width 0.1524) (layer GND) (net 0))
   (segment (start 262.41609 63.25896) (end 263.82472 63.25896) (width 0.1524) (layer GND) (net 0))
   (segment (start 261.28472 63.25896) (end 262.41609 63.25896) (width 0.1524) (layer GND) (net 0))
   (segment (start 264.95609 63.25896) (end 266.36472 63.25896) (width 0.1524) (layer GND) (net 0))
   (segment (start 263.82472 63.25896) (end 264.95609 63.25896) (width 0.1524) (layer GND) (net 0))
-  (via (at 272.18982 43.367422) (size 0.6096) (drill 0.3048) (layers F.Cu GND) (net 0))
+  (via (at 269.11046 65.12814) (size 0.6096) (drill 0.3048) (layers F.Cu GND) (net 4))
+  (via (at 270.30172 56.52262) (size 0.6096) (drill 0.3048) (layers F.Cu GND) (net 4))
   (segment (start 272.186422 21.213542) (end 268.11732 21.213542) (width 0.1524) (layer F.Cu) (net 1))
   (segment (start 273.80184 22.27656) (end 273.24944 22.27656) (width 0.1524) (layer F.Cu) (net 1))
@@
   (via (at 242.23472 79.3496) (size 0.6096) (drill 0.3048) (layers F.Cu GND) (net 4))
   (via (at 229.05212 67.8688) (size 0.6096) (drill 0.3048) (layers F.Cu GND) (net 4))
-  (via (at 277.79472 56.72836) (size 0.6096) (drill 0.3048) (layers F.Cu GND) (net 4))
   (via (at 243.0272 42.04208) (size 0.6096) (drill 0.3048) (layers F.Cu GND) (net 4))
   (segment (start 243.014313 44.322947) (end 243.014313 42.054967) (width 0.1524) (layer F.Cu) (net 4))
@@
   (via (at 275.263021 78.890541) (size 0.6096) (drill 0.3048) (layers F.Cu GND) (net 4))
   (segment (start 275.25472 75.49896) (end 275.25472 78.88224) (width 0.1524) (layer GND) (net 4))
+  (via (at 266.95908 56.58866) (size 0.6096) (drill 0.3048) (layers F.Cu GND) (net 4))
+  (segment (start 270.37538 56.44896) (end 270.30172 56.52262) (width 0.1524) (layer F.Cu) (net 4))
+  (segment (start 267.02512 56.52262) (end 266.95908 56.58866) (width 0.1524) (layer F.Cu) (net 4))
+  (segment (start 270.30172 56.52262) (end 267.02512 56.52262) (width 0.1524) (layer F.Cu) (net 4))
+  (segment (start 269.415259 65.432939) (end 269.11046 65.12814) (width 0.1524) (layer F.Cu) (net 4))
+  (segment (start 270.454119 66.471799) (end 269.415259 65.432939) (width 0.1524) (layer F.Cu) (net 4))
+  (segment (start 270.454119 69.377561) (end 270.454119 66.471799) (width 0.1524) (layer F.Cu) (net 4))
+  (segment (start 270.14932 69.68236) (end 270.454119 69.377561) (width 0.1524) (layer F.Cu) (net 4))
   (segment (start 254.280232 94.629968) (end 253.027832 94.629968) (width 0.1524) (layer F.Cu) (net 5))
   (segment (start 256.157832 94.629968) (end 254.280232 94.629968) (width 0.1524) (layer F.Cu) (net 5))
